File: kicad/PSU/PSU.kicad_sch (KiCad schematic)
At the start: 43 parts, among them J1 B2B-PH-K-S, J2 Output Header, U1 BQ21040DBVR, U2 RT4812GJ8F, U3 AP3445LW6-7, U4 AP3445LW6-7

Commit message: Added Fuses & USB-C data to PSU
Parts:
- removed J2: Output Header, Connector_JST:JST_EH_B7B-EH-A_1x07_P2.50mm_Vertical, symbol Connector:Conn_01x07_Pin
- added F1, F2, F3, F4: 2A, symbol Device:Fuse_Small
- added J2: Conn_01x09_Pin, symbol Connector:Conn_01x09_Pin
- R2, R4: value 5.1K -> 22K
Connections:
- net +1.8V: now also F2.2; no longer C10.2, C12.1, C9.2, L3.1, R13.2
- net +3.3V: now also F3.2; no longer C11.1, C7.2, C8.2, L2.1, R12.2
- net +5V: now also F4.2; no longer C5.2, C6.1, R6.1, U2.3 (VOUT)
- net 1.8V: now also J2.9 (Pin_9)
- net 3.3V: now also J2.8 (Pin_8)
- net 5V: now also J2.7 (Pin_7)
- net GND: now also J2.6 (Pin_6)
- net PG_1.8: now also J2.5 (Pin_5)
- net PG_3.3: now also J2.4 (Pin_4)
- net Vbat: now also F1.1; no longer J1.1
- net at R8.2, R9.1: now also J2.3 (Pin_3)
- net D+: now reaches USB-C1.A6 (DP1)
- net D+: now also USB-C1.B6 (DP2), J2.2 (Pin_2)
- net D-: now reaches USB-C1.A7 (DN1)
- net D-: now also USB-C1.B7 (DN2), J2.1 (Pin_1)
- new net: C11.1, C7.2, C8.2, F3.1, L2.1, R12.2
- new net: C10.2, C12.1, C9.2, F2.1, L3.1, R13.2
- new net: C5.2, C6.1, F4.1, R6.1, U2.3 (VOUT)
- new net: F1.2, J1.1
- no-connect marks 6 -> 2
Other:
- moved on the sheet: R2, R4
