File: kicad/mcu-board/mcu-board.kicad_sch (KiCad schematic)
At the start: 44 parts, among them J12 UJ20-C-H-G-SMT-P16-TR, J3 5015680407, J4 5015680407, J5 5015680407, J6 Conn_01x07, SW1 SW_Push, SW2 SW_Push, U1 Lora1276-C1-868, U2 ESP32-S3-WROOM-1U-N16R8

Commit message: feat: finished pcb, might add more artwork later?
Parts:
- removed J3, J4, J5: 5015680407, CONN_5015680000-SD_04_MOL, symbol 2026-01-26_05-30-52:5015680407
- removed J6: Conn_01x07, symbol Connector_Generic:Conn_01x07
- removed R13, R14: 22, symbol Device:R
- removed TP11: TestPoint, TestPoint:TestPoint_Pad_D1.0mm, symbol Connector:TestPoint
- added C4: 0.1uf, Capacitor_SMD:C_0805_2012Metric, symbol Device:C
- added J1: Conn_01x03, Connector_PinHeader_2.54mm:PinHeader_1x03_P2.54mm_Vertical, symbol Connector_Generic:Conn_01x03
- added J2: Conn_01x02, Connector_PinHeader_2.54mm:PinHeader_1x02_P2.54mm_Vertical, symbol Connector_Generic:Conn_01x02
- added J3, J4, J5: 533980471, PSAT_Library:MOLEX_533980471, symbol PSAT_Library:533980471
- added TP1, TP10, TP20, TP23, TP7, TP8, TP9: TestPoint, TestPoint:TestPoint_Pad_D1.0mm, symbol Connector:TestPoint
- R1, R2, R3, R4: value 4.7k -> 5.1k
- SW1, SW2: footprint Button_Switch_SMD:SW_Push_1P1T_NO_CK_KMR2 -> Button_Switch_SMD:SW_Tactile_SPST_NO_Straight_CK_PTS636Sx25SMTRLFS
- U2: footprint PSAT_Library:XCVR_ESP32-S3-WROOM-1U-N16R8 -> footprints2:ESP32-S3-WROOM-1U; Availability (none) -> In Stock; Check_prices (none) -> https://www.snapeda.com/parts/ESP32-S3-WROOM-1U-N16R8/Espre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; Description_1 (none) -> Bluetooth, WiFi 802.11b/g/n, Bluetooth v5.0 Transceiver Mod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; MF (none) -> Espressif Systems; MP (none) -> ESP32-S3-WROOM-1U-N16R8; Package (none) -> SMD-41 Espressif Systems; Price (none) -> None; SnapEDA_Link (none) -> https://www.snapeda.com/parts/ESP32-S3-WROOM-1U-N16R8/Espre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
- renumbered C7 to C1, C1 to C2, C9 to C3, C10 to C5, C2 to C6, C8 to C7, J12 to J6, R11 to R5, R5 to R6, R6 to R7, TP4 to TP11, TP5 to TP12, TP6 to TP13, TP7 to TP14, TP9 to TP15, TP8 to TP16, TP12 to TP17, TP13 to TP18, TP17 to TP19, TP15 to TP3, TP3 to TP4, TP16 to TP5, TP1 to TP6, TP10 to VBAT1
Connections:
- net I2CEXT1_SDA is gone; now on net I2C1_SDA_IO41: R2.1, TP3.1
- net LIGHT_1 is gone; now on net I2C1_SCL_IO40: U2.33 (IO40)
- net BUZ_GND: now also J1.3 (Pin_3), TP23.1
- net D+: now also U2.14 (IO20)
- net D-: now also U2.13 (IO19)
- net GND: now also C4.2, J1.1 (Pin_1)
- net BUZZER renamed CAM_IO21
- net CAM_IO21: now also J5.3
- net CAM_IO10 renamed LORA_SPI3_CLK_IO10
- net LORA_SPI3_CLK_IO10: now also U1.4 (SCK), TP9.1
- net CAM_IO38 renamed BUZZER_IO38
- net CAM_IO39 renamed IO39
- net IO39: now also J2.1 (Pin_1)
- net CAM_IO9 renamed LORA_IRQ_IO9
- net LORA_IRQ_IO9: now also TP16.1, U1.14 (DI0)
- net GPIO45 renamed IO45
- net IO45: now also J2.2 (Pin_2)
- net GPIO46 renamed LORA_SPI3_CS_IO46
- net LORA_SPI3_CS_IO46: now also U1.5 (~{SS}), TP10.1
- net GPIO47 renamed CAM_IO47
- net CAM_IO47: now also J5.4
- net GPIO48 renamed SERVO_IO48
- net SERVO_IO48: now also TP6.1, J1.2 (Pin_2)
- net GPS_U1RX_IO42 renamed LIGHT_1_IO42
- net LIGHT_1_IO42: now also J4.3
- net GPS_U1TX_IO41 renamed I2C1_SDA_IO41
- net I2C1_SDA_IO41: now also J4.2
- net I2C0_SCL_IO11 renamed LORA_SPI3_D_IO11
- net LORA_SPI3_D_IO11: now also U1.3 (MOSI), TP8.1
- net I2C0_SDA_IO12 renamed LORA_SPI3_Q_IO12
- net LORA_SPI3_Q_IO12: now also U1.2 (MISO), TP7.1
- net I2C1_SCL_IO13 renamed CAM_IO13
- net CAM_IO13: now also J5.1
- net I2C1_SDA_IO14 renamed CAM_IO14
- net CAM_IO14: now also J5.2
- net I2CEXT0_SCL renamed I2C0_SCL_IO4
- net I2C0_SCL_IO4: now also U2.4 (IO4), J3.1
- net I2CEXT0_SDA renamed I2C0_SDA_IO5
- net I2C0_SDA_IO5: now also U2.5 (IO5), J3.2
- net I2CEXT1_SCL renamed I2C1_SCL_IO40
- net I2C1_SCL_IO40: now also J4.1
- net LIGHT2_ADC1CH1 renamed LIGHT_2_ADC1CH1_IO2
- net LIGHT_2_ADC1CH1_IO2: now also J4.4
- removed net LORA_IRQ_IO16: TP16.1, U1.14 (DI0), U2.9 (IO16)
- net LORA_SPI3_CLK renamed ~{LORA_EN}_IO3
- net ~{LORA_EN}_IO3: now also U1.6 (~{RESET}), TP1.1; no longer U1.4 (SCK)
- removed net LORA_SPI3_CS0: U1.5 (~{SS}), U2.4 (IO4), U2.5 (IO5)
- net LORA_SPI3_D renamed GPS_U1TX_IO6
- net GPS_U1TX_IO6: now also J3.3; no longer U1.3 (MOSI)
- net LORA_SPI3_Q renamed GPS_U1RX_IO7
- net GPS_U1RX_IO7: now also J3.4; no longer U1.2 (MISO)
- net POWER_ST: no longer names the net of U2.10 (IO17)
- net SERVO_IO8: no longer names the net of U2.12 (IO8)
- net SERVO_IO8: no longer TP6.1
- net V_BAT renamed VBAT_IO1
- net VBAT_IO1: now also C4.1
- net ~{LORA_EN}_IO15: no longer names the net of U2.8 (IO15)
- net ~{LORA_EN}_IO15: no longer U1.6 (~{RESET})
- new net Power Management/POWER_ST: TP20.1
- no-connect marks 10 -> 20
Other:
- sheet Buzzer Power renamed BUZZER_IO38 Power
- sheet BUZZER_IO38 Power ports: added none; removed GND
- sheet Power Management ports: added VBAT_IO1; removed V_BAT
- note added: "Can use [46, 48] normally, as not the R16 variant"
- note added: "Sensor I2C 1 And GPS uart"
- note added: "Sensor I2C 2 and light sensors"
- note added: "[IO35, IO37] are used for internal PSRAM"
- note removed: "Can use normally, as not the R16 variant"
- note removed: "GPS Uart"
- note removed: "IO35 ~ IO37 (inclusive) are used for internal PSRAM"
- note removed: "Place close to chip"
- note removed: "Power state (Optional?) For determining current power source."
- note removed: "Sensor I2C 1"
- note removed: "Sensor I2C 2"
- moved on the sheet: AE1, C2, C3, TP11, TP12, TP13, TP14, TP15, TP16, TP17, TP18, TP19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
